File: io.kicad_sch (KiCad schematic)
At the start: 17 parts, among them J7 JUMP_vdd, J8 JUMP_gnd, SW1 SW_Push, SW2 SW_Push1, SW3 SW_Push2, SW4 SW_Push3, SW5 SW_Push

Commit message: v1.0
Connections:
- net VSS renamed GND
Changed lines of the file:
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@@
     (pin "2")
+  )
+  (symbol (lib_id "power:GND") (at 240.03 66.04 0) (unit 1)
+    (in_bom yes) (on_board yes) (fields_autoplaced)
+    (property "Reference" "#PWR017" (id 0) (at 240.03 72.39 0)
+      (effects (font (size 1.27 1.27)) hide)
+    )
+    (property "Value" "GND" (id 1) (at 240.03 71.12 0))
+    (property "Footprint" "" (id 2) (at 240.03 66.04 0)
+      (effects (font (size 1.27 1.27)) hide)
+    )
+    (property "Datasheet" "" (id 3) (at 240.03 66.04 0)
+      (effects (font (size 1.27 1.27)) hide)
+    )
+    (pin "1")
   )
   (symbol (lib_id "power:VDD") (at 161.29 26.67 0) (unit 1)
@@
     )
     (property "Datasheet" "" (id 3) (at 161.29 26.67 0)
-      (effects (font (size 1.27 1.27)) hide)
-    )
-    (pin "1")
-  )
-  (symbol (lib_id "power:VSS") (at 26.67 60.96 0) (mirror x) (unit 1)
-    (in_bom yes) (on_board yes) (fields_autoplaced)
-    (property "Reference" "#PWR013" (id 0) (at 26.67 57.15 0)
-      (effects (font (size 1.27 1.27)) hide)
-    )
-    (property "Value" "VSS" (id 1) (at 26.67 66.04 0))
-    (property "Footprint" "" (id 2) (at 26.67 60.96 0)
-      (effects (font (size 1.27 1.27)) hide)
-    )
-    (property "Datasheet" "" (id 3) (at 26.67 60.96 0)
       (effects (font (size 1.27 1.27)) hide)
     )
@@
     (pin "2")
   )
+  (symbol (lib_id "power:GND") (at 187.96 62.23 0) (unit 1)
+    (in_bom yes) (on_board yes) (fields_autoplaced)
+    (property "Reference" "#PWR015" (id 0) (at 187.96 68.58 0)
+      (effects (font (size 1.27 1.27)) hide)
+    )
+    (property "Value" "GND" (id 1) (at 187.96 67.31 0))
+    (property "Footprint" "" (id 2) (at 187.96 62.23 0)
+      (effects (font (size 1.27 1.27)) hide)
+    )
+    (property "Datasheet" "" (id 3) (at 187.96 62.23 0)
+      (effects (font (size 1.27 1.27)) hide)
+    )
+    (pin "1")
+  )
   (symbol (lib_id "Device:R") (at 161.29 38.1 0) (unit 1)
     (in_bom yes) (on_board yes) (fields_autoplaced)
@@
     (pin "2")
   )
-  (symbol (lib_id "power:VSS") (at 240.03 66.04 0) (mirror x) (unit 1)
-    (in_bom yes) (on_board yes) (fields_autoplaced)
-    (property "Reference" "#PWR025" (id 0) (at 240.03 62.23 0)
-      (effects (font (size 1.27 1.27)) hide)
-    )
-    (property "Value" "VSS" (id 1) (at 240.03 71.12 0))
-    (property "Footprint" "" (id 2) (at 240.03 66.04 0)
-      (effects (font (size 1.27 1.27)) hide)
-    )
-    (property "Datasheet" "" (id 3) (at 240.03 66.04 0)
+  (symbol (lib_id "power:GND") (at 93.98 63.5 0) (unit 1)
+    (in_bom yes) (on_board yes) (fields_autoplaced)
+    (property "Reference" "#PWR013" (id 0) (at 93.98 69.85 0)
+      (effects (font (size 1.27 1.27)) hide)
+    )
+    (property "Value" "GND" (id 1) (at 93.98 68.58 0))
+    (property "Footprint" "" (id 2) (at 93.98 63.5 0)
+      (effects (font (size 1.27 1.27)) hide)
+    )
+    (property "Datasheet" "" (id 3) (at 93.98 63.5 0)
       (effects (font (size 1.27 1.27)) hide)
     )
@@
     (pin "1")
   )
-  (symbol (lib_id "power:VSS") (at 187.96 62.23 0) (mirror x) (unit 1)
-    (in_bom yes) (on_board yes) (fields_autoplaced)
-    (property "Reference" "#PWR021" (id 0) (at 187.96 58.42 0)
-      (effects (font (size 1.27 1.27)) hide)
-    )
-    (property "Value" "VSS" (id 1) (at 187.96 67.31 0))
-    (property "Footprint" "" (id 2) (at 187.96 62.23 0)
-      (effects (font (size 1.27 1.27)) hide)
-    )
-    (property "Datasheet" "" (id 3) (at 187.96 62.23 0)
-      (effects (font (size 1.27 1.27)) hide)
-    )
-    (pin "1")
-  )
   (symbol (lib_id "Switch:SW_Push") (at 111.76 60.96 0) (unit 1)
     (in_bom yes) (on_board yes) (fields_autoplaced)
@@
     (pin "2")
   )
-  (symbol (lib_id "power:VSS") (at 93.98 63.5 0) (mirror x) (unit 1)
-    (in_bom yes) (on_board yes) (fields_autoplaced)
-    (property "Reference" "#PWR017" (id 0) (at 93.98 59.69 0)
-      (effects (font (size 1.27 1.27)) hide)
-    )
-    (property "Value" "VSS" (id 1) (at 93.98 68.58 0))
-    (property "Footprint" "" (id 2) (at 93.98 63.5 0)
-      (effects (font (size 1.27 1.27)) hide)
-    )
-    (property "Datasheet" "" (id 3) (at 93.98 63.5 0)
-      (effects (font (size 1.27 1.27)) hide)
-    )
+  (symbol (lib_id "power:GND") (at 26.67 60.96 0) (unit 1)
+    (in_bom yes) (on_board yes) (fields_autoplaced)
+    (property "Reference" "#PWR012" (id 0) (at 26.67 67.31 0)
+      (effects (font (size 1.27 1.27)) hide)
+    )
+    (property "Value" "GND" (id 1) (at 26.67 66.04 0))
+    (property "Footprint" "" (id 2) (at 26.67 60.96 0)
+      (effects (font (size 1.27 1.27)) hide)
+    )
+    (property "Datasheet" "" (id 3) (at 26.67 60.96 0)
+      (effects (font (size 1.27 1.27)) hide)
+    )

Commit message: v3.1 all
Parts:
- SW1, SW2, SW3, SW4, SW5: footprint Library:SW_Push_6x3.6mm_H2.5mm -> Library2:SW_Push_6x3.6mm_H2.5mm
Changed lines of the file:
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@@
 (kicad_sch (version 20211123) (generator eeschema)
   (paper "A4")
+  (title_block
+    (date "2022-09-12")
+    (rev "soy")
+  )
   (junction (at 187.96 59.69) (diameter 0) (color 0 0 0 0)
   )
@@
     (property "Reference" "SW4" (id 0) (at 111.76 67.31 0))
     (property "Value" "SW_Push3" (id 1) (at 111.76 69.85 0))
-    (property "Footprint" "Library:SW_Push_6x3.6mm_H2.5mm" (id 2) (at 111.76 69.85 0)
+    (property "Footprint" "Library2:SW_Push_6x3.6mm_H2.5mm" (id 2) (at 111.76 69.85 0)
       (effects (font (size 1.27 1.27)) hide)
     )
@@
     (property "Reference" "SW3" (id 0) (at 111.76 53.34 0))
     (property "Value" "SW_Push2" (id 1) (at 111.76 55.88 0))
-    (property "Footprint" "Library:SW_Push_6x3.6mm_H2.5mm" (id 2) (at 111.76 55.88 0)
+    (property "Footprint" "Library2:SW_Push_6x3.6mm_H2.5mm" (id 2) (at 111.76 55.88 0)
       (effects (font (size 1.27 1.27)) hide)
     )
@@
     (property "Reference" "SW1" (id 0) (at 111.76 29.21 0))
     (property "Value" "SW_Push" (id 1) (at 111.76 31.75 0))
-    (property "Footprint" "Library:SW_Push_6x3.6mm_H2.5mm" (id 2) (at 111.76 31.75 0)
+    (property "Footprint" "Library2:SW_Push_6x3.6mm_H2.5mm" (id 2) (at 111.76 31.75 0)
       (effects (font (size 1.27 1.27)) hide)
     )
@@
     (property "Reference" "SW2" (id 0) (at 111.76 40.64 0))
     (property "Value" "SW_Push1" (id 1) (at 111.76 43.18 0))
-    (property "Footprint" "Library:SW_Push_6x3.6mm_H2.5mm" (id 2) (at 111.76 43.18 0)
+    (property "Footprint" "Library2:SW_Push_6x3.6mm_H2.5mm" (id 2) (at 111.76 43.18 0)
       (effects (font (size 1.27 1.27)) hide)
     )
@@
     (property "Reference" "SW5" (id 0) (at 176.53 44.45 0))
     (property "Value" "SW_Push" (id 1) (at 176.53 46.99 0))
-    (property "Footprint" "Library:SW_Push_6x3.6mm_H2.5mm" (id 2) (at 176.53 46.99 0)
-      (effects (font (size 1.27 1.27)) hide)
-    )
+    (property "Footprint" "Library2:SW_Push_6x3.6mm_H2.5mm" (id 2) (at 176.53 46.99 0)
+      (effects (font (size 1.27 1.27)) hide)
+    )
