File: jtag.kicad_sch (KiCad schematic)
At the start: 6 parts, among them J4 Conn_ARM_JTAG_SWD_20

Commit message: v1.0
Connections:
- net VSS renamed GND
Changed lines of the file:
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@@
     (pin "2")
-  )
-  (symbol (lib_id "power:VSS") (at 111.76 109.22 0) (mirror x) (unit 1)
-    (in_bom yes) (on_board yes) (fields_autoplaced)
-    (property "Reference" "#PWR015" (id 0) (at 111.76 105.41 0)
-      (effects (font (size 1.27 1.27)) hide)
-    )
-    (property "Value" "VSS" (id 1) (at 111.76 114.3 0))
-    (property "Footprint" "" (id 2) (at 111.76 109.22 0)
-      (effects (font (size 1.27 1.27)) hide)
-    )
-    (property "Datasheet" "" (id 3) (at 111.76 109.22 0)
-      (effects (font (size 1.27 1.27)) hide)
-    )
-    (pin "1")
   )
   (symbol (lib_id "Device:R") (at 171.45 66.04 0) (mirror x) (unit 1)
@@
       (effects (font (size 1.27 1.27)) hide)
     )
+    (pin "1")
+  )
+  (symbol (lib_id "power:GND") (at 111.76 109.22 0) (unit 1)
+    (in_bom yes) (on_board yes) (fields_autoplaced)
+    (property "Reference" "#PWR020" (id 0) (at 111.76 115.57 0)
+      (effects (font (size 1.27 1.27)) hide)
+    )
+    (property "Value" "GND" (id 1) (at 111.76 114.3 0))
+    (property "Footprint" "" (id 2) (at 111.76 109.22 0)
+      (effects (font (size 1.27 1.27)) hide)
+    )
+    (property "Datasheet" "" (id 3) (at 111.76 109.22 0)
+      (effects (font (size 1.27 1.27)) hide)
+    )
