File: msm2.kicad_sch (KiCad schematic)
At the start: 13 parts, among them J10 Conn_01x36, J11 Conn_01x36, J12 Conn_01x36, J9 Conn_01x36, U1 STM32F407ZETx, Y1 25M, Y2 32.768k

Commit message: v1.0
Connections:
- net VSS is gone; now on net GND: C1.1, C2.1, C22.1, C23.1, C24.1, C25.1, U1.107 (VSS), U1.120 (VSS), U1.130 (VSS), U1.16 (VSS), U1.31 (VSSA), U1.38 (VSS), U1.51 (VSS), U1.61 (VSS), U1.83 (VSS), U1.94 (VSS), Y1.2, Y1.4
- net BOOT0: now also J11.30 (Pin_30)
- net RESET: now also J12.25 (Pin_25)
- net VDD: now also J10.16 (Pin_16), J10.26 (Pin_26), J10.3 (Pin_3), J10.36 (Pin_36), J11.13 (Pin_13), J11.23 (Pin_23), J11.35 (Pin_35), J11.36 (Pin_36), J12.17 (Pin_17), J12.30 (Pin_30), J12.32 (Pin_32), J12.33 (Pin_33), J9.12 (Pin_12), J9.23 (Pin_23), J9.36 (Pin_36)
- net Vb: now also J12.6 (Pin_6)
- net GND: now reaches J11.12 (Pin_12)
- net GND: now also J10.15 (Pin_15), J10.2 (Pin_2), J10.25 (Pin_25), J11.22 (Pin_22), J12.16 (Pin_16), J12.31 (Pin_31), J9.11 (Pin_11), J9.22 (Pin_22), J9.35 (Pin_35)
- no-connect marks 32 -> 4

Commit message: good pcb
Connections:
- net PC14: no longer J12.8 (Pin_8)
- net PC15: no longer J12.9 (Pin_9)
- no-connect marks 4 -> 6
Changed lines of the file:
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@@
   (junction (at 127 196.85) (diameter 0) (color 0 0 0 0)
   )
+  (no_connect (at 251.46 111.76))
+  (no_connect (at 251.46 114.3))
   (no_connect (at 251.46 149.86))
   (no_connect (at 251.46 152.4))
@@
     (effects (font (size 1.27 1.27)) (justify left bottom))
   )
-  (label "PC14" (at 251.46 111.76 180)
-    (effects (font (size 1.27 1.27)) (justify right bottom))
-  )
   (label "PF11" (at 20.32 36.83 180)
     (effects (font (size 1.27 1.27)) (justify right bottom))
@@
     (effects (font (size 1.27 1.27)) (justify right bottom))
   )
-  (label "PC15" (at 251.46 114.3 180)
-    (effects (font (size 1.27 1.27)) (justify right bottom))
-  )

Commit message: v3.1 all
Other:
- title: (none) -> STM32F429ZGT6
Changed lines of the file:
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@@
 (kicad_sch (version 20211123) (generator eeschema)
   (paper "A4")
+  (title_block
+    (title "STM32F429ZGT6")
+    (date "2022-09-12")
+    (rev "soy")
+  )
   (junction (at 129.54 196.85) (diameter 0) (color 0 0 0 0)
   )
@@
     )
     (path "/9b5c3b29-0ba0-4e2e-bed2-763180cc28b9/a31cf181-fe02-4f9f-9cfd-0a272d6ec767"
-      (reference "SW1") (unit 1) (value "SW_Push") (footprint "Library:SW_Push_6x3.6mm_H2.5mm")
+      (reference "SW1") (unit 1) (value "SW_Push") (footprint "Library2:SW_Push_6x3.6mm_H2.5mm")
     )
     (path "/9b5c3b29-0ba0-4e2e-bed2-763180cc28b9/dbc4401d-0309-4a07-8d57-5cf981052a92"
-      (reference "SW2") (unit 1) (value "SW_Push1") (footprint "Library:SW_Push_6x3.6mm_H2.5mm")
+      (reference "SW2") (unit 1) (value "SW_Push1") (footprint "Library2:SW_Push_6x3.6mm_H2.5mm")
     )
     (path "/9b5c3b29-0ba0-4e2e-bed2-763180cc28b9/94e6013f-d911-4c17-8901-d4baf3928eff"
-      (reference "SW3") (unit 1) (value "SW_Push2") (footprint "Library:SW_Push_6x3.6mm_H2.5mm")
+      (reference "SW3") (unit 1) (value "SW_Push2") (footprint "Library2:SW_Push_6x3.6mm_H2.5mm")
     )
     (path "/9b5c3b29-0ba0-4e2e-bed2-763180cc28b9/38e9997a-d55c-4a5f-917f-5c7384be3f79"
-      (reference "SW4") (unit 1) (value "SW_Push3") (footprint "Library:SW_Push_6x3.6mm_H2.5mm")
+      (reference "SW4") (unit 1) (value "SW_Push3") (footprint "Library2:SW_Push_6x3.6mm_H2.5mm")
     )
     (path "/9b5c3b29-0ba0-4e2e-bed2-763180cc28b9/f45209b4-fc10-46eb-bdf5-94061622ad4c"
-      (reference "SW5") (unit 1) (value "SW_Push") (footprint "Library:SW_Push_6x3.6mm_H2.5mm")
+      (reference "SW5") (unit 1) (value "SW_Push") (footprint "Library2:SW_Push_6x3.6mm_H2.5mm")
     )
     (path "/6d9ae86f-8faa-459d-8f87-32364671ad9f"
