File: power.kicad_sch (KiCad schematic)
At the start: 23 parts, among them J1 PowerH, J2 PowerL, J3 USB_vcc, U2 AMS1117-3.3

Commit message: v1.0
Parts:
- added C27: 1uF, Capacitor_SMD:C_0603_1608Metric_Pad1.08x0.95mm_HandSolder, symbol Device:C_Small
Connections:
- net GND: now also C27.2
- net VDD: now also C27.1
Changed lines of the file:
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@@
   (junction (at 156.21 127) (diameter 0) (color 0 0 0 0)
   )
+  (junction (at 214.63 127) (diameter 0) (color 0 0 0 0)
+  )
   (junction (at 156.21 132.08) (diameter 0) (color 0 0 0 0)
   )
@@
   (junction (at 50.8 40.64) (diameter 0) (color 0 0 0 0)
   )
+  (junction (at 123.19 132.08) (diameter 0) (color 0 0 0 0)
+  )
+  (junction (at 100.33 132.08) (diameter 0) (color 0 0 0 0)
+  )
+  (junction (at 93.98 80.01) (diameter 0) (color 0 0 0 0)
+  )
+  (junction (at 139.7 127) (diameter 0) (color 0 0 0 0)
+  )
+  (junction (at 214.63 132.08) (diameter 0) (color 0 0 0 0)
+  )
+  (junction (at 115.57 132.08) (diameter 0) (color 0 0 0 0)
+  )
+  (junction (at 132.08 132.08) (diameter 0) (color 0 0 0 0)
+  )
+  (junction (at 63.5 40.64) (diameter 0) (color 0 0 0 0)
+  )
+  (junction (at 110.49 58.42) (diameter 0) (color 0 0 0 0)
+  )
+  (junction (at 139.7 132.08) (diameter 0) (color 0 0 0 0)
+  )
+  (junction (at 204.47 132.08) (diameter 0) (color 0 0 0 0)
+  )
+  (junction (at 123.19 127) (diameter 0) (color 0 0 0 0)
+  )
+  (junction (at 148.59 127) (diameter 0) (color 0 0 0 0)
+  )
   (junction (at 93.98 87.63) (diameter 0) (color 0 0 0 0)
-  )
-  (junction (at 63.5 43.18) (diameter 0) (color 0 0 0 0)
-  )
-  (junction (at 123.19 132.08) (diameter 0) (color 0 0 0 0)
-  )
-  (junction (at 100.33 132.08) (diameter 0) (color 0 0 0 0)
-  )
-  (junction (at 93.98 80.01) (diameter 0) (color 0 0 0 0)
-  )
-  (junction (at 139.7 127) (diameter 0) (color 0 0 0 0)
-  )
-  (junction (at 115.57 132.08) (diameter 0) (color 0 0 0 0)
-  )
-  (junction (at 132.08 132.08) (diameter 0) (color 0 0 0 0)
-  )
-  (junction (at 63.5 40.64) (diameter 0) (color 0 0 0 0)
-  )
-  (junction (at 110.49 58.42) (diameter 0) (color 0 0 0 0)
-  )
-  (junction (at 139.7 132.08) (diameter 0) (color 0 0 0 0)
-  )
-  (junction (at 204.47 132.08) (diameter 0) (color 0 0 0 0)
-  )
-  (junction (at 123.19 127) (diameter 0) (color 0 0 0 0)
-  )
-  (junction (at 148.59 127) (diameter 0) (color 0 0 0 0)
   )
   (junction (at 179.07 45.72) (diameter 0) (color 0 0 0 0)
@@
     (stroke (width 0) (type default) (color 0 0 0 0))
   )
-  (wire (pts (xy 179.07 55.88) (xy 179.07 58.42))
-    (stroke (width 0) (type default) (color 0 0 0 0))
-  )
   (wire (pts (xy 187.96 127) (xy 196.85 127))
     (stroke (width 0) (type default) (color 0 0 0 0))
@@
     (stroke (width 0) (type default) (color 0 0 0 0))
   )
-  (wire (pts (xy 68.58 43.18) (xy 63.5 43.18))
-    (stroke (width 0) (type default) (color 0 0 0 0))
-  )
   (wire (pts (xy 115.57 132.08) (xy 123.19 132.08))
     (stroke (width 0) (type default) (color 0 0 0 0))
   )
+  (wire (pts (xy 214.63 132.08) (xy 223.52 132.08))
+    (stroke (width 0) (type default) (color 0 0 0 0))
+  )
   (wire (pts (xy 148.59 132.08) (xy 156.21 132.08))
     (stroke (width 0) (type default) (color 0 0 0 0))
@@
     (stroke (width 0) (type default) (color 0 0 0 0))
   )
-  (wire (pts (xy 63.5 43.18) (xy 63.5 44.45))
-    (stroke (width 0) (type default) (color 0 0 0 0))
-  )
   (wire (pts (xy 156.21 132.08) (xy 156.21 139.7))
     (stroke (width 0) (type default) (color 0 0 0 0))
@@
     (stroke (width 0) (type default) (color 0 0 0 0))
   )
-  (wire (pts (xy 68.58 44.45) (xy 68.58 43.18))
-    (stroke (width 0) (type default) (color 0 0 0 0))
-  )
   (wire (pts (xy 50.8 40.64) (xy 50.8 38.1))
     (stroke (width 0) (type default) (color 0 0 0 0))
@@
     (stroke (width 0) (type default) (color 0 0 0 0))
   )
+  (wire (pts (xy 214.63 127) (xy 223.52 127))
+    (stroke (width 0) (type default) (color 0 0 0 0))
+  )
   (wire (pts (xy 189.23 44.45) (xy 189.23 45.72))
     (stroke (width 0) (type default) (color 0 0 0 0))
@@
     (stroke (width 0) (type default) (color 0 0 0 0))
   )
-  (wire (pts (xy 63.5 40.64) (xy 63.5 43.18))
+  (wire (pts (xy 63.5 40.64) (xy 63.5 46.99))
     (stroke (width 0) (type default) (color 0 0 0 0))
   )
@@
   )
   (wire (pts (xy 165.1 127) (xy 172.72 127))
-    (stroke (width 0) (type default) (color 0 0 0 0))
-  )
-  (wire (pts (xy 93.98 87.63) (xy 93.98 88.9))
     (stroke (width 0) (type default) (color 0 0 0 0))
   )
@@
     (pin "2")
   )
-  (symbol (lib_id "power:VSS") (at 156.21 139.7 0) (mirror x) (unit 1)
-    (in_bom yes) (on_board yes) (fields_autoplaced)
-    (property "Reference" "#PWR011" (id 0) (at 156.21 135.89 0)
-      (effects (font (size 1.27 1.27)) hide)
-    )
-    (property "Value" "VSS" (id 1) (at 156.21 144.78 0))
-    (property "Footprint" "" (id 2) (at 156.21 139.7 0)
-      (effects (font (size 1.27 1.27)) hide)
-    )
-    (property "Datasheet" "" (id 3) (at 156.21 139.7 0)
+  (symbol (lib_id "Device:C_Small") (at 223.52 129.54 0) (unit 1)
+    (in_bom yes) (on_board yes) (fields_autoplaced)
+    (property "Reference" "C27" (id 0) (at 226.06 128.2762 0)
+      (effects (font (size 1.27 1.27)) (justify left))
+    )
+    (property "Value" "1uF" (id 1) (at 226.06 130.8162 0))
+    (property "Footprint" "Capacitor_SMD:C_0603_1608Metric_Pad1.08x0.95mm_HandSolder" (id 2) (at 223.52 129.54 0)
+      (effects (font (size 1.27 1.27)) hide)
+    )
+    (property "Datasheet" "~" (id 3) (at 223.52 129.54 0)
+      (effects (font (size 1.27 1.27)) hide)
+    )
+    (pin "1")
+    (pin "2")
+  )
+  (symbol (lib_id "power:GND") (at 93.98 87.63 0) (unit 1)
+    (in_bom yes) (on_board yes) (fields_autoplaced)
+    (property "Reference" "#PWR06" (id 0) (at 93.98 93.98 0)
+      (effects (font (size 1.27 1.27)) hide)
+    )
+    (property "Value" "GND" (id 1) (at 93.98 92.71 0))
+    (property "Footprint" "" (id 2) (at 93.98 87.63 0)
+      (effects (font (size 1.27 1.27)) hide)
+    )
+    (property "Datasheet" "" (id 3) (at 93.98 87.63 0)
       (effects (font (size 1.27 1.27)) hide)
     )
@@
     (pin "1")
     (pin "2")
-  )
-  (symbol (lib_id "power:VSS") (at 179.07 58.42 0) (mirror x) (unit 1)
-    (in_bom yes) (on_board yes) (fields_autoplaced)
-    (property "Reference" "#PWR012" (id 0) (at 179.07 54.61 0)
-      (effects (font (size 1.27 1.27)) hide)
-    )
-    (property "Value" "VSS" (id 1) (at 179.07 63.5 0))
-    (property "Footprint" "" (id 2) (at 179.07 58.42 0)
-      (effects (font (size 1.27 1.27)) hide)
-    )
-    (property "Datasheet" "" (id 3) (at 179.07 58.42 0)
-      (effects (font (size 1.27 1.27)) hide)
-    )
-    (pin "1")
-  )
-  (symbol (lib_id "power:VSS") (at 63.5 44.45 0) (mirror x) (unit 1)
-    (in_bom yes) (on_board yes) (fields_autoplaced)
-    (property "Reference" "#PWR06" (id 0) (at 63.5 40.64 0)
-      (effects (font (size 1.27 1.27)) hide)
-    )
-    (property "Value" "VSS" (id 1) (at 63.5 49.53 0))
-    (property "Footprint" "" (id 2) (at 63.5 44.45 0)
-      (effects (font (size 1.27 1.27)) hide)
-    )
-    (property "Datasheet" "" (id 3) (at 63.5 44.45 0)
-      (effects (font (size 1.27 1.27)) hide)
-    )
-    (pin "1")
   )
   (symbol (lib_id "Device:C_Small") (at 132.08 129.54 0) (unit 1)
@@
     (pin "1")
   )
-  (symbol (lib_id "power:GND") (at 68.58 44.45 0) (unit 1)
-    (in_bom yes) (on_board yes) (fields_autoplaced)
-    (property "Reference" "#PWR029" (id 0) (at 68.58 50.8 0)
-      (effects (font (size 1.27 1.27)) hide)
-    )
-    (property "Value" "GND" (id 1) (at 68.58 49.53 0))
-    (property "Footprint" "" (id 2) (at 68.58 44.45 0)
-      (effects (font (size 1.27 1.27)) hide)
-    )
-    (property "Datasheet" "" (id 3) (at 68.58 44.45 0)
+  (symbol (lib_id "power:GND") (at 63.5 46.99 0) (unit 1)
+    (in_bom yes) (on_board yes) (fields_autoplaced)
+    (property "Reference" "#PWR029" (id 0) (at 63.5 53.34 0)
+      (effects (font (size 1.27 1.27)) hide)
+    )
+    (property "Value" "GND" (id 1) (at 63.5 52.07 0))
+    (property "Footprint" "" (id 2) (at 63.5 46.99 0)
+      (effects (font (size 1.27 1.27)) hide)
+    )
+    (property "Datasheet" "" (id 3) (at 63.5 46.99 0)
       (effects (font (size 1.27 1.27)) hide)
     )
@@
     (pin "2")
   )
+  (symbol (lib_id "power:GND") (at 156.21 139.7 0) (unit 1)
+    (in_bom yes) (on_board yes) (fields_autoplaced)
+    (property "Reference" "#PWR08" (id 0) (at 156.21 146.05 0)
+      (effects (font (size 1.27 1.27)) hide)
+    )
+    (property "Value" "GND" (id 1) (at 156.21 144.78 0))
+    (property "Footprint" "" (id 2) (at 156.21 139.7 0)
+      (effects (font (size 1.27 1.27)) hide)
+    )
+    (property "Datasheet" "" (id 3) (at 156.21 139.7 0)
+      (effects (font (size 1.27 1.27)) hide)
+    )
+    (pin "1")
+  )
   (symbol (lib_id "Device:C_Small") (at 214.63 129.54 0) (unit 1)
     (in_bom yes) (on_board yes) (fields_autoplaced)
@@
     )
     (property "Datasheet" "" (id 3) (at 124.46 58.42 0)
+      (effects (font (size 1.27 1.27)) hide)
+    )
+    (pin "1")
+  )
+  (symbol (lib_id "power:GND") (at 179.07 55.88 0) (unit 1)
+    (in_bom yes) (on_board yes) (fields_autoplaced)
+    (property "Reference" "#PWR011" (id 0) (at 179.07 62.23 0)
+      (effects (font (size 1.27 1.27)) hide)
+    )
+    (property "Value" "GND" (id 1) (at 179.07 60.96 0))
+    (property "Footprint" "" (id 2) (at 179.07 55.88 0)
+      (effects (font (size 1.27 1.27)) hide)
+    )
+    (property "Datasheet" "" (id 3) (at 179.07 55.88 0)
       (effects (font (size 1.27 1.27)) hide)
     )
@@
     (pin "2")
   )
-  (symbol (lib_id "power:VSS") (at 93.98 88.9 0) (mirror x) (unit 1)
-    (in_bom yes) (on_board yes) (fields_autoplaced)
-    (property "Reference" "#PWR08" (id 0) (at 93.98 85.09 0)
-      (effects (font (size 1.27 1.27)) hide)
-    )
-    (property "Value" "VSS" (id 1) (at 93.98 93.98 0))
-    (property "Footprint" "" (id 2) (at 93.98 88.9 0)
-      (effects (font (size 1.27 1.27)) hide)
-    )
-    (property "Datasheet" "" (id 3) (at 93.98 88.9 0)
-      (effects (font (size 1.27 1.27)) hide)
-    )
-    (pin "1")
-  )
   (symbol (lib_id "Device:C_Small") (at 156.21 129.54 0) (unit 1)
