File: usart.kicad_sch (KiCad schematic)
At the start: 6 parts, among them J5 usb_new, J6 JUMP_usb, U3 CH340C

Commit message: v1.0
Connections:
- net VSS renamed GND
Changed lines of the file:
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@@
     (pin "9")
   )
-  (symbol (lib_id "power:VSS") (at 95.25 99.06 0) (mirror x) (unit 1)
+  (symbol (lib_id "power:GND") (at 144.78 96.52 0) (unit 1)
     (in_bom yes) (on_board yes) (fields_autoplaced)
-    (property "Reference" "#PWR020" (id 0) (at 95.25 95.25 0)
+    (property "Reference" "#PWR023" (id 0) (at 144.78 102.87 0)
       (effects (font (size 1.27 1.27)) hide)
     )
-    (property "Value" "VSS" (id 1) (at 95.25 104.14 0))
+    (property "Value" "GND" (id 1) (at 144.78 101.6 0))
+    (property "Footprint" "" (id 2) (at 144.78 96.52 0)
+      (effects (font (size 1.27 1.27)) hide)
+    )
+    (property "Datasheet" "" (id 3) (at 144.78 96.52 0)
+      (effects (font (size 1.27 1.27)) hide)
+    )
+    (pin "1")
+  )
+  (symbol (lib_id "power:GND") (at 95.25 99.06 0) (unit 1)
+    (in_bom yes) (on_board yes) (fields_autoplaced)
+    (property "Reference" "#PWR021" (id 0) (at 95.25 105.41 0)
+      (effects (font (size 1.27 1.27)) hide)
+    )
+    (property "Value" "GND" (id 1) (at 95.25 104.14 0))
     (property "Footprint" "" (id 2) (at 95.25 99.06 0)
       (effects (font (size 1.27 1.27)) hide)
@@
     (pin "1")
     (pin "2")
-  )
-  (symbol (lib_id "power:VSS") (at 148.59 57.15 0) (mirror x) (unit 1)
-    (in_bom yes) (on_board yes) (fields_autoplaced)
-    (property "Reference" "#PWR028" (id 0) (at 148.59 53.34 0)
-      (effects (font (size 1.27 1.27)) hide)
-    )
-    (property "Value" "VSS" (id 1) (at 148.59 62.23 0))
-    (property "Footprint" "" (id 2) (at 148.59 57.15 0)
-      (effects (font (size 1.27 1.27)) hide)
-    )
-    (property "Datasheet" "" (id 3) (at 148.59 57.15 0)
-      (effects (font (size 1.27 1.27)) hide)
-    )
-    (pin "1")
   )
   (symbol (lib_id "Device:LED") (at 125.73 93.98 270) (mirror x) (unit 1)
@@
     (pin "2")
   )
+  (symbol (lib_id "power:GND") (at 148.59 57.15 0) (unit 1)
+    (in_bom yes) (on_board yes) (fields_autoplaced)
+    (property "Reference" "#PWR025" (id 0) (at 148.59 63.5 0)
+      (effects (font (size 1.27 1.27)) hide)
+    )
+    (property "Value" "GND" (id 1) (at 148.59 62.23 0))
+    (property "Footprint" "" (id 2) (at 148.59 57.15 0)
+      (effects (font (size 1.27 1.27)) hide)
+    )
+    (property "Datasheet" "" (id 3) (at 148.59 57.15 0)
+      (effects (font (size 1.27 1.27)) hide)
+    )
+    (pin "1")
+  )
   (symbol (lib_id "New_Library:usb_new") (at 95.25 73.66 0) (unit 1)
     (in_bom yes) (on_board yes) (fields_autoplaced)
@@
       (effects (font (size 1.27 1.27)) hide)
     )
-    (pin "1")
-  )
-  (symbol (lib_id "power:VSS") (at 144.78 96.52 0) (mirror x) (unit 1)
-    (in_bom yes) (on_board yes) (fields_autoplaced)
-    (property "Reference" "#PWR023" (id 0) (at 144.78 92.71 0)
-      (effects (font (size 1.27 1.27)) hide)
-    )
-    (property "Value" "VSS" (id 1) (at 144.78 101.6 0))
-    (property "Footprint" "" (id 2) (at 144.78 96.52 0)
-      (effects (font (size 1.27 1.27)) hide)
-    )
-    (property "Datasheet" "" (id 3) (at 144.78 96.52 0)
-      (effects (font (size 1.27 1.27)) hide)
-    )
