File: msm2.kicad_pcb (KiCad board)
At the start: 2 copper layers, 150 x 100 mm, 66 parts, among them J1 PowerH, J10 Conn_01x36, J11 Conn_01x36, J12 Conn_01x36, J2 PowerL, J3 USB_vcc, J4 Conn_ARM_JTAG_SWD_20, J5 usb_new, J6 JUMP_usb, J7 JUMP_vdd, J8 JUMP_gnd, J9 Conn_01x36, SW1 SW_Push, SW2 SW_Push1, SW3 SW_Push2, SW4 SW_Push3, SW5 SW_Push, U1 STM32F407ZETx, U2 AMS1117-3.3, U3 CH340C, Y1 25M, Y2 32.768k

Commit message: good pcb
Parts:
- moved C14 48.3 mm to (106.5, 35.9), turned to -90 degrees
- moved D3 11.3 mm to (3.77, 89.6), turned to 0 degrees
- moved R3 4.50 mm to (9.81, 89.7), turned to 180 degrees
- moved D4 3.25 mm to (144.7, 51.8)
- moved R10 2.92 mm to (144.6, 54.7)
- moved SW1 1.91 mm to (12.1, 84.0)
- moved C17 1.24 mm to (104.8, 35.9), turned to -90 degrees
- moved J7 1.23 mm to (137.2, 67.3)
- moved C21 1.06 mm to (10.3, 75.1)
- moved R9 0.70 mm to (14.2, 75.1)
- moved R5 0.50 mm to (90.1, 10.5)
Connections:
- J12 pad 8: /PC14 -> unconnected-(J12-Pad8)
- J12 pad 9: /PC15 -> unconnected-(J12-Pad9)
Routing:
- net BOOT0: track 53.1 -> 126.0 mm, vias 1 -> 4
- net RESET: track 89.9 -> 152.7 mm, vias 1 -> 4
- net GND: track 189.0 -> 219.1 mm, vias 31 -> 37
- net VDD: track 682.1 -> 710.6 mm
- net unconnected-(J3-Pad6): track 0.00 -> 12.6 mm
- net Net-(J6-Pad2): track 10.4 -> 7.29 mm
- net Net-(D3-Pad2): track 2.65 -> 4.29 mm
- net /PA0: track 85.6 -> 87.1 mm
- net /PF8: track 95.4 -> 96.7 mm
- net Net-(J7-Pad3): track 7.20 -> 8.43 mm
- net Net-(J7-Pad4): track 7.10 -> 8.32 mm
- net /PF10: track 80.3 -> 79.3 mm, vias 1 -> 3
- net /PD10: track 48.5 -> 47.7 mm
- net /PF9: track 77.5 -> 78.1 mm, vias 1 -> 3
- net Net-(D4-Pad2): track 3.52 -> 2.93 mm
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Other:
- outline, holes or cut-outs redrawn

Commit message: pcb v2.0
Parts:
- added REF**: WEEE-Logo_8.4x12mm_SilkScreen, Symbol:WEEE-Logo_8.4x12mm_SilkScreen, F.Cu at (144.2, 87.8)
- added REF**: KiCad-Logo2_6mm_SilkScreen, Symbol:KiCad-Logo2_6mm_SilkScreen, B.Cu at (11.5, 13.2)
- added REF**: ESD-Logo_8.9x8mm_SilkScreen, Symbol:ESD-Logo_8.9x8mm_SilkScreen, B.Cu at (139.0, 89.3)
Routing:
- net /PE3: track 88.7 -> 89.7 mm
- net GND: track 219.1 -> 218.4 mm, vias 37 -> 41
Other:
- board text added: "+"
- board text added: "10"
- board text added: "15"
- board text added: "20"
- board text added: "2022.9.12"
- board text added: "25"
- board text added: "30"
- board text added: "35"
- board text added: "5"
- board text added: "BOOT0"
- board text added: "BOOT1"
- board text added: "Boot1"
- board text added: "GND"
- board text added: "H+"
- board text added: "L+"
- board text added: "PA0"
- board text added: "PA1"
- board text added: "PA10"
- board text added: "PA11"
- board text added: "PA12"
- board text added: "PA13"
- board text added: "PA14"
- board text added: "PA15"
- board text added: "PA2"
- board text added: "PA3"
- board text added: "PA4"
- board text added: "PA5"
- board text added: "PA6"
- board text added: "PA7"
- board text added: "PA8"
- board text added: "PA9"
- board text added: "PB0"
- board text added: "PB1"
- board text added: "PB10"
- board text added: "PB11"
- board text added: "PB12"
- board text added: "PB13"
- board text added: "PB14"
- board text added: "PB15"
- board text added: "PB3"
- board text added: "PB4"
- board text added: "PB5"
- board text added: "PB6"
- board text added: "PB7"
- board text added: "PB8"
- board text added: "PB9"
- board text added: "PC0"
- board text added: "PC1"
- board text added: "PC10"
- board text added: "PC11"
- board text added: "PC12"
- board text added: "PC13"
- board text added: "PC2"
- board text added: "PC3"
- board text added: "PC4"
- board text added: "PC5"
- board text added: "PC6"
- board text added: "PC7"
- board text added: "PC8"
- board text added: "PC9"
- board text added: "PD0"
- board text added: "PD1"
- board text added: "PD10"
- board text added: "PD11"
- board text added: "PD12"
- board text added: "PD13"
- board text added: "PD14"
- board text added: "PD15"
- board text added: "PD2"
- board text added: "PD3"
- board text added: "PD4"
- board text added: "PD5"
- board text added: "PD6"
- board text added: "PD7"
- board text added: "PD8"
- board text added: "PD9"
- board text added: "PE0"
- board text added: "PE1"
- board text added: "PE10"
- board text added: "PE11"
- board text added: "PE12"
- board text added: "PE13"
- board text added: "PE14"
- board text added: "PE15"
- board text added: "PE2"
- board text added: "PE3"
- board text added: "PE4"
- board text added: "PE5"
- board text added: "PE6"
- board text added: "PE7"
- board text added: "PE8"
- board text added: "PE9"
- board text added: "PF0"
- board text added: "PF1"
- board text added: "PF10"
- board text added: "PF11"
- board text added: "PF12"
- board text added: "PF13"
- board text added: "PF14"
- board text added: "PF15"
- board text added: "PF2"
- board text added: "PF3"
- board text added: "PF4"
- board text added: "PF5"
- board text added: "PF6"
- board text added: "PF7"
- board text added: "PF8"
- board text added: "PF9"
- board text added: "PG0"
- board text added: "PG1"
- board text added: "PG10"
- board text added: "PG11"
- board text added: "PG12"
- board text added: "PG13"
- board text added: "PG14"
- board text added: "PG15"
- board text added: "PG2"
- board text added: "PG3"
- board text added: "PG4"
- board text added: "PG5"
- board text added: "PG6"
- board text added: "PG7"
- board text added: "PG8"
- board text added: "PG9"
- board text added: "RESET"
- board text added: "STM32F429ZGT6"
- board text added: "VDD"
- board text added: "Vb"
- board text added: "WK_UP"

Commit message: pcb v3.0
Parts:
- moved R7 39.2 mm to (103.2, 7.80)
- moved R4 26.2 mm to (93.3, 4.80)
- moved R6 23.7 mm to (37.2, 4.80), turned to 180 degrees
- moved R8 19.0 mm to (37.1, 7.50), turned to 180 degrees
- moved R5 14.1 mm to (103.1, 5.10)
Routing:
- net /PB3: track 63.6 -> 85.4 mm, vias 0 -> 1
- net /PB4: track 53.3 -> 72.8 mm
- net VDD: track 710.6 -> 725.1 mm
- net GND: track 218.4 -> 214.7 mm
- net /PA14: track 91.2 -> 93.4 mm, vias 1 -> 4
- net /PA15: track 91.9 -> 93.3 mm
- net /PA13: track 122.6 -> 122.5 mm, vias 1 -> 2
Other:
- board text added: "SWCLK"
- board text added: "SWDIO"
- board text added: "SWO"

Commit message: pcb v3.1
Parts:
- moved D1 2.40 mm to (15.3, 61.0)
- moved SW4 2.31 mm to (12.6, 21.5)
- moved D2 2.29 mm to (15.3, 64.2)
- moved SW3 1.33 mm to (12.7, 16.0)
- moved J10 1.31 mm to (36.3, 96.3)
Routing:
- net VDD: track 725.1 -> 712.9 mm
- net /PE3: track 89.7 -> 97.7 mm
- net /PC3: track 73.1 -> 67.0 mm
- net /PA2: track 77.5 -> 83.3 mm
- net /PC2: track 71.8 -> 66.2 mm
- net /PD4: track 31.9 -> 26.7 mm
- net /PA1: track 76.8 -> 81.8 mm
- net /PD5: track 32.3 -> 27.6 mm
- net /PB14: track 55.5 -> 60.1 mm
- net /PD3: track 31.6 -> 27.0 mm
- net /PE2: track 81.0 -> 85.4 mm
- net /PA0: track 87.1 -> 91.3 mm
- net /PD2: track 30.9 -> 27.8 mm
- net /PC1: track 67.9 -> 65.2 mm
- net BOOT1: track 127.7 -> 130.2 mm
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Other:
- outline, holes or cut-outs redrawn

Commit message: v3.3
Parts:
- removed the REF** at (144.2, 87.8)
- added REF**: MountingHole_3.2mm_M3_DIN965_Pad, MountingHole:MountingHole_3.2mm_M3_DIN965_Pad, F.Cu at (5.00, 95.0)
- added REF**: WEEE-Logo_5.6x8mm_SilkScreen, Symbol:WEEE-Logo_5.6x8mm_SilkScreen, F.Cu at (145.1, 86.9)
- added REF**: MountingHole_2.2mm_M2_DIN965_Pad, MountingHole:MountingHole_2.2mm_M2_DIN965_Pad, F.Cu at (39.0, 23.0)
- added REF**: MountingHole_3.2mm_M3_DIN965_Pad, MountingHole:MountingHole_3.2mm_M3_DIN965_Pad, F.Cu at (145.0, 95.0)
- added REF**: MountingHole_2.2mm_M2_DIN965_Pad, MountingHole:MountingHole_2.2mm_M2_DIN965_Pad, F.Cu at (109.0, 23.0)
- added REF**: MountingHole_3.2mm_M3_DIN965_Pad, MountingHole:MountingHole_3.2mm_M3_DIN965_Pad, F.Cu at (145.0, 5.00)
- added REF**: MountingHole_2.2mm_M2_DIN965_Pad, MountingHole:MountingHole_2.2mm_M2_DIN965_Pad, F.Cu at (31.2, 94.7)
- added REF**: MountingHole_3.2mm_M3_DIN965_Pad, MountingHole:MountingHole_3.2mm_M3_DIN965_Pad, F.Cu at (5.00, 5.00)
- added REF**: MountingHole_2.2mm_M2_DIN965_Pad, MountingHole:MountingHole_2.2mm_M2_DIN965_Pad, F.Cu at (126.6, 88.0)
- moved REF** 1.43 mm to (138.1, 88.2)
Other:
- outline, holes or cut-outs redrawn
